File: buildbutton2/buildbutton.sch (KiCad schematic (older format))
At the start: 17 parts, among them J1 BATTERY, J2 IO0, J3 BUTTON, J4 LED, J5 USB, Q1 IRLIZ44N, U1 S7V8F3, U2 U3V12F9, U3 ESP32_DATA, U4 ESP_UART

Commit message: BuildButton v3
Other:
- moved on the sheet: C_BLK1, C_PWR1
Changed lines of the file:
@@
 L GND #PWR08
 U 1 1 5A4DAA0C
-P 4000 4950
-F 0 "#PWR08" H 4000 4700 50  0001 C CNN
-F 1 "GND" H 4000 4800 50  0000 C CNN
-F 2 "" H 4000 4950 50  0001 C CNN
-F 3 "" H 4000 4950 50  0001 C CNN
-	1    4000 4950
+P 3950 4800
+F 0 "#PWR08" H 3950 4550 50  0001 C CNN
+F 1 "GND" H 3950 4650 50  0000 C CNN
+F 2 "" H 3950 4800 50  0001 C CNN
+F 3 "" H 3950 4800 50  0001 C CNN
+	1    3950 4800
 	1    0    0    -1
 $EndComp
@@
 L C C_BLK1
 U 1 1 5A4DAAF7
-P 4000 4650
-F 0 "C_BLK1" H 4025 4750 50  0000 L CNN
-F 1 "100uF" H 4025 4550 50  0000 L CNN
-F 2 "Capacitors_SMD:CP_Elec_6.3x7.7" H 4038 4500 50  0001 C CNN
-F 3 "" H 4000 4650 50  0001 C CNN
-	1    4000 4650
+P 3950 4500
+F 0 "C_BLK1" H 3975 4600 50  0000 L CNN
+F 1 "100uF" H 3975 4400 50  0000 L CNN
+F 2 "Capacitors_SMD:CP_Elec_6.3x7.7" H 3988 4350 50  0001 C CNN
+F 3 "" H 3950 4500 50  0001 C CNN
+	1    3950 4500
 	1    0    0    -1
 $EndComp
@@
 L C C_PWR1
 U 1 1 5A4DABDE
-P 4500 4650
-F 0 "C_PWR1" H 4525 4750 50  0000 L CNN
-F 1 "100nF" H 4525 4550 50  0000 L CNN
-F 2 "Capacitors_THT:C_Disc_D5.0mm_W2.5mm_P2.50mm" H 4538 4500 50  0001 C CNN
-F 3 "" H 4500 4650 50  0001 C CNN
-	1    4500 4650
+P 4450 4500
+F 0 "C_PWR1" H 4475 4600 50  0000 L CNN
+F 1 "100nF" H 4475 4400 50  0000 L CNN
+F 2 "Capacitors_THT:C_Disc_D5.0mm_W2.5mm_P2.50mm" H 4488 4350 50  0001 C CNN
+F 3 "" H 4450 4500 50  0001 C CNN
+	1    4450 4500
 	1    0    0    -1
 $EndComp
 Wire Wire Line
-	4000 4200 4000 4500
+	3950 4050 3950 4350
 Wire Wire Line
-	4000 4450 4500 4450
+	3950 4300 4450 4300
 Wire Wire Line
-	4500 4450 4500 4500
-Connection ~ 4000 4450
+	4450 4300 4450 4350
+Connection ~ 3950 4300
 Wire Wire Line
-	4000 4800 4000 4950
+	3950 4650 3950 4800
 Wire Wire Line
-	4000 4850 4500 4850
+	3950 4700 4450 4700
 Wire Wire Line
-	4500 4850 4500 4800
-Connection ~ 4000 4850
+	4450 4700 4450 4650
+Connection ~ 3950 4700
 Wire Wire Line
 	2700 4100 2500 4100
@@
 	1    0    0    -1
 $EndComp
-Text GLabel 3850 4200 0    60   Input ~ 0
+Text GLabel 3800 4050 0    60   Input ~ 0
 3V3
 Wire Wire Line
-	3850 4200 4000 4200
+	3800 4050 3950 4050
 Text GLabel 2450 3450 0    60   Input ~ 0
 3V3
