File: buildbutton3/buildbutton.sch (KiCad schematic (older format))
At the start: 17 parts, among them J1 BATTERY, J2 IO0, J3 BUTTON, J4 LED, J5 USB, Q1 IRLIZ44N, U1 S7V8F3, U2 U3V12F9, U3 ESP32_DATA, U4 ESP_UART

Commit message: BuildButton v3
Parts:
- removed J5: USB, Socket_Strips:Socket_Strip_Angled_1x04_Pitch2.54mm, symbol USB
- removed U1: S7V8F3, pololu:S7V8F3, symbol S7V8F3
- added C_IN1, C_OUT1: 10uF, Capacitors_Tantalum_SMD:CP_Tantalum_Case-A_EIA-3216-18_Reflow, symbol C
- added J5: PROG, Socket_Strips:Socket_Strip_Angled_1x06_Pitch2.54mm, symbol PROG
- added U1: LM1117-3.3, TO_SOT_Packages_SMD:SOT-223, symbol LM1117-3.3
- C_EN1, C_IO0: value 1nF -> 2.2nF; footprint Capacitors_THT:C_Disc_D5.0mm_W2.5mm_P2.50mm -> Capacitors_SMD:C_1206
- C_PWR1: footprint Capacitors_THT:C_Disc_D5.0mm_W2.5mm_P2.50mm -> Capacitors_Tantalum_SMD:CP_Tantalum_Case-A_EIA-3216-18_Reflow
- J4: footprint TerminalBlocks_Phoenix:TerminalBlock_Phoenix_PT-3.5mm_2pol -> Socket_Strips:Socket_Strip_Angled_1x02_Pitch2.54mm
- Q1: value IRLIZ44N -> IRLL014N; footprint TO_SOT_Packages_SMD:TO-252-2 -> TO_SOT_Packages_SMD:SOT-223
- U2: value U3V12F9 -> U3V12F5
Connections:
- net 3V3: now also C_OUT1.1, J5.1 (Pin_1), U1.2 (VO)
- net EN: now also J5.5 (Pin_5)
- net GND: now also C_IN1.2, C_OUT1.2, J5.4 (Pin_4), U1.1 (GND); no longer U2.2 (GND)
- net VCC: now also C_IN1.1, U1.3 (VI)
- net at U4.4 (TX): now also J5.2 (Pin_2)
- net at U4.5 (RX): now also J5.3 (Pin_3)
- net IO0: now reaches C_IO0.1, J2.1 (Pin_1), R_IO0.2
- net IO0: now also J5.6 (Pin_6)
- net at J4.2 (Pin_2), Q1.2 (D): now also U2.2 (GND)
- net 9V: no longer names the net of J4.1 (Pin_1), U2.3 (VOUT)
Other:
- moved on the sheet: J1, J3, J4, Q1, R_BTN1, U2, U3, U4

Commit message: Buildbutton3 update
Parts:
- U2: symbol U3V12F9 -> U3V12F9-RESCUE-buildbutton
Changed lines of the file:
@@
 EESchema Schematic File Version 2
+LIBS:buildbutton-rescue
 LIBS:power
 LIBS:device
@@
 LIBS:contrib
 LIBS:valves
+LIBS:dominik
+LIBS:ncp1402
 LIBS:pololu
-LIBS:ncp1402
-LIBS:dominik
 LIBS:buildbutton-cache
 EELAYER 25 0
@@
 $EndComp
 $Comp
-L U3V12F9 U2
+L U3V12F9-RESCUE-buildbutton U2
 U 1 1 5A4D6211
 P 4100 2800
