File: pms5003-lopy/pms5003.sch (KiCad schematic (older format))
At the start: 23 parts, among them J1 Battery, J2 DS3231, J3 PMS5003, J4 SHT10, J5 P2, J6 PROG, J7 USB_OTG, Q1 IRF540N, Q2 IRF7309IPBF, U1 U3V12F5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

Commit message: Add a pull-up resistor to RTC_VCC
Parts:
- added R7: 100, Resistors_SMD:R_1206, symbol R
- J3: symbol PMS5003 -> PMS5003-RESCUE-pms5003
Connections:
- net PMS_EN: now also U11.6 (P4); no longer U11.21 (P19)
- net SHT_RTC_VCC: now also U11.21 (P19), R7.2; no longer U11.6 (P4)
- net 3V3: now reaches U11.26 (3.3v)
- net 3V3: now also R7.1
- no-connect marks 17 -> 16
Other:
- moved on the sheet: Q2A, R4, R5, R6
Changed lines of the file:
@@
 EESchema Schematic File Version 2
+LIBS:pms5003-rescue
 LIBS:power
 LIBS:device
@@
 $EndComp
 $Comp
-L PMS5003 J3
+L PMS5003-RESCUE-pms5003 J3
 U 1 1 5A61FE04
 P 1800 2350
@@
 Wire Wire Line
 	4300 1950 4500 1950
-Text GLabel 4500 2100 2    60   Input ~ 0
-PMS_EN
+Text GLabel 4750 2100 2    60   Input ~ 0
+SHT_RTC_VCC
 $Comp
 L PWR_FLAG #FLG09
@@
 	2500 1200 2650 1200
 Wire Wire Line
-	4500 2100 4300 2100
+	4300 2100 4750 2100
 Wire Wire Line
 	3800 3550 3450 3550
@@
 L IRF7309IPBF Q2
 U 1 1 5A64A830
-P 6100 2300
-F 0 "Q2" H 6350 2375 50  0000 L CNN
-F 1 "IRF7309IPBF" H 6350 2300 50  0000 L CNN
-F 2 "Housings_SOIC:SO-8_5.3x6.2mm_Pitch1.27mm" H 6350 2225 50  0001 L CNN
-F 3 "" H 6100 2300 50  0001 L CNN
-	1    6100 2300
+P 6550 2300
+F 0 "Q2" H 6800 2375 50  0000 L CNN
+F 1 "IRF7309IPBF" H 6800 2300 50  0000 L CNN
+F 2 "Housings_SOIC:SO-8_5.3x6.2mm_Pitch1.27mm" H 6800 2225 50  0001 L CNN
+F 3 "" H 6550 2300 50  0001 L CNN
+	1    6550 2300
 	1    0    0    -1
 $EndComp
@@
 Wire Wire Line
 	4550 2550 4300 2550
-Text GLabel 5300 2350 0    60   Input ~ 0
+Text GLabel 5750 2350 0    60   Input ~ 0
 ADC_EN
 Wire Wire Line
-	5800 2350 5900 2350
+	6250 2350 6350 2350
 $Comp
 L GND #PWR014
 U 1 1 5A64AF40
-P 6200 2600
-F 0 "#PWR014" H 6200 2350 50  0001 C CNN
-F 1 "GND" H 6200 2450 50  0000 C CNN
-F 2 "" H 6200 2600 50  0001 C CNN
-F 3 "" H 6200 2600 50  0001 C CNN
-	1    6200 2600
-	1    0    0    -1
-$EndComp
-Wire Wire Line
-	6200 2600 6200 2500
+P 6650 2600
+F 0 "#PWR014" H 6650 2350 50  0001 C CNN
+F 1 "GND" H 6650 2450 50  0000 C CNN
+F 2 "" H 6650 2600 50  0001 C CNN
+F 3 "" H 6650 2600 50  0001 C CNN
+	1    6650 2600
+	1    0    0    -1
+$EndComp
+Wire Wire Line
+	6650 2600 6650 2500
 $Comp
 L R R5
 U 1 1 5A64AFEE
-P 6200 1800
-F 0 "R5" V 6280 1800 50  0000 C CNN
-F 1 "47k" V 6200 1800 50  0000 C CNN
-F 2 "Resistors_SMD:R_1206" V 6130 1800 50  0001 C CNN
-F 3 "" H 6200 1800 50  0001 C CNN
-	1    6200 1800
+P 6650 1800
+F 0 "R5" V 6730 1800 50  0000 C CNN
+F 1 "47k" V 6650 1800 50  0000 C CNN
+F 2 "Resistors_SMD:R_1206" V 6580 1800 50  0001 C CNN
+F 3 "" H 6650 1800 50  0001 C CNN
+	1    6650 1800
 	1    0    0    -1
 $EndComp
@@
 L R R4
 U 1 1 5A64B0D7
-P 6200 1400
-F 0 "R4" V 6280 1400 50  0000 C CNN
-F 1 "100k" V 6200 1400 50  0000 C CNN
-F 2 "Resistors_SMD:R_1206" V 6130 1400 50  0001 C CNN
-F 3 "" H 6200 1400 50  0001 C CNN
-	1    6200 1400
-	1    0    0    -1
-$EndComp
-Wire Wire Line
-	6200 1950 6200 2100
-Wire Wire Line
-	6200 1550 6200 1650
-Wire Wire Line
-	6200 1000 6200 1250
-Wire Wire Line
-	6200 1600 6400 1600
-Connection ~ 6200 1600
-Text GLabel 6400 1600 2    60   Input ~ 0
+P 6650 1400
+F 0 "R4" V 6730 1400 50  0000 C CNN
+F 1 "100k" V 6650 1400 50  0000 C CNN
+F 2 "Resistors_SMD:R_1206" V 6580 1400 50  0001 C CNN
+F 3 "" H 6650 1400 50  0001 C CNN
+	1    6650 1400
+	1    0    0    -1
+$EndComp
+Wire Wire Line
+	6650 1950 6650 2100
+Wire Wire Line
+	6650 1550 6650 1650
+Wire Wire Line
+	6650 1000 6650 1250
+Wire Wire Line
+	6650 1600 6850 1600
+Connection ~ 6650 1600
+Text GLabel 6850 1600 2    60   Input ~ 0
 ADC
-NoConn ~ 6300 2100
+NoConn ~ 6750 2100
 $Comp
 L MAX1811 U2
@@
 NoConn ~ 1250 5550
 NoConn ~ 850  5750
-Text GLabel 6100 1000 0    60   Input ~ 0
+Text GLabel 6550 1000 0    60   Input ~ 0
 VBATT+
 Wire Wire Line
-	6100 1000 6200 1000
+	6550 1000 6650 1000
 $Comp
 L R R6
 U 1 1 5A65B0A2
-P 5650 2350
-F 0 "R6" V 5730 2350 50  0000 C CNN
-F 1 "100" V 5650 2350 50  0000 C CNN
-F 2 "Resistors_SMD:R_1206" V 5580 2350 50  0001 C CNN
-F 3 "" H 5650 2350 50  0001 C CNN
-	1    5650 2350
+P 6100 2350
+F 0 "R6" V 6180 2350 50  0000 C CNN
+F 1 "100" V 6100 2350 50  0000 C CNN
+F 2 "Resistors_SMD:R_1206" V 6030 2350 50  0001 C CNN
+F 3 "" H 6100 2350 50  0001 C CNN
+	1    6100 2350
 	0    -1   -1   0
 $EndComp
 Wire Wire Line
-	5500 2350 5300 2350
+	5950 2350 5750 2350
 Text GLabel 2500 1800 0    60   Input ~ 0
-SHT_RTC_VCC
+PMS_EN
 Wire Wire Line
 	2650 1800 2500 1800
-NoConn ~ 4300 1350
+Text GLabel 4500 1350 2    60   Input ~ 0
+3V3
+Text GLabel 4900 2250 2    60   Input ~ 0
+3V3
+$Comp
+L R R7
+U 1 1 5A6A6EEE
+P 4650 2250
+F 0 "R7" V 4730 2250 50  0000 C CNN
+F 1 "100" V 4650 2250 50  0000 C CNN
+F 2 "Resistors_SMD:R_1206" V 4580 2250 50  0001 C CNN
+F 3 "" H 4650 2250 50  0001 C CNN
+	1    4650 2250
+	0    1    1    0
+$EndComp
+Wire Wire Line
+	4400 2100 4400 2250
+Wire Wire Line
+	4400 2250 4500 2250
+Connection ~ 4400 2100
+Wire Wire Line
+	4800 2250 4900 2250
+Wire Wire Line
+	4500 1350 4300 1350
 $EndSCHEMATC
