File: pms5003-lopy/v2/pms5003.kicad_pcb (KiCad board)
At the start: 2 copper layers, 73 x 75 mm, 26 parts, among them J1 Battery, J2 DISPLAY, J3 PMS5003, J5 P2, J6 PROG, J7 USB_OTG, Q1 IRF7309IPBF, Q2 IRF7309IPBF, U1 U3V12F5, U11 LoPy4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

Commit message: Fixes to v2 PMS5003
Parts:
- J5: footprint Socket_Strips:Socket_Strip_Straight_1x02_Pitch2.54mm -> Pin_Headers:Pin_Header_Straight_1x02_Pitch2.54mm
- J6: footprint Socket_Strips:Socket_Strip_Straight_1x04_Pitch2.54mm -> Pin_Headers:Pin_Header_Straight_1x04_Pitch2.54mm
