File: pms5003-lopy/v2/pms5003.sch (KiCad schematic (older format))
At the start: 23 parts, among them J1 Battery, J2 DISPLAY, J3 PMS5003, J5 P2, J6 PROG, J7 USB_OTG, Q1 IRF7309IPBF, Q2 IRF7309IPBF, U1 U3V12F5, U11 LoPy4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

Commit message: Fixes to v2 PMS5003
Connections:
- net 3V3: no longer J2.5 (Pin_5)
- net GND: now also J2.5 (Pin_5)
Changed lines of the file:
@@
 LIBS:contrib
 LIBS:valves
-LIBS:pycom
 LIBS:pololu
 LIBS:dominik
@@
 CLK
 Text GLabel 6100 2500 0    60   Input ~ 0
-3V3
+GND
 Text GLabel 6100 2650 0    60   Input ~ 0
 DC
