File: pms5003-lopy/v1/pms5003.sch (KiCad schematic (older format))
At the start: 24 parts, among them J1 Battery, J2 DS3231, J3 PMS5003, J4 SHT10, J5 P2, J6 PROG, J7 USB_OTG, Q1 IRF540N, Q2 IRF7309IPBF, U1 U3V12F5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

Commit message: Update to KiCad 5
Parts:
- J7: symbol USB_OTG -> USB_OTG-RESCUE-pms5003
Changed lines of the file:
@@
 LIBS:contrib
 LIBS:valves
-LIBS:pycom
-LIBS:pololu
-LIBS:dominik
 LIBS:pms5003-cache
 EELAYER 25 0
@@
 $EndComp
 $Comp
-L USB_OTG J7
+L USB_OTG-RESCUE-pms5003 J7
 U 1 1 5A6513FA
 P 950 5350
